File: Hardware/Kicad/Laster/012-Amesis-ColdSartE85/012-Amesis-ColdSartE85.kicad_pcb (KiCad board)
At the start: 2 copper layers, 52.1 x 26.5 mm, 8 parts, among them J1 Screw_Terminal_01x02, J2 Conn_01x05_Female, J3 Conn_01x03_Female

Commit message: maj
Parts:
- added  : LOGO, AP_Amesis Logo:AmesisProject Logo 15mm, F.Cu at (106.8, 52.7)
- added G***: LOGO, AP_Amesis Logo:KiCad QR Code La Boutique Amesis Project, F.Cu at (115.9, 59.3)
Other:
- board text added: "1"
- board text added: "12v"
- board text added: "2"
- board text added: "3"
- board text added: "5V"
- board text added: "Amesis_ColdStartE85_v0.01"
- board text added: "Arduino Nano"
- board text added: "G2"
- board text added: "G2 = To Cluster G62 = To ECU"
- board text added: "G62"
- board text added: "GND"
- board text added: "Gnd"
- board text added: "IAT"
- board text added: "InPut IAT"
- board text added: "JP"
- board text added: "Jumper Option Jumper 1&2 = +++ No Jumper = ++ Jumper 2&3 = +"
- board text added: "OutPut to ECU"
- board text added: "X9C103S"

Commit message: maj
Parts:
- removed the G*** at (115.9, 59.3)
- added G***: LOGO, AP_Amesis Logo:10x10 KiCad QR Code La Boutique Amesis Project, F.Cu at (114.1, 56.6)
- added G***: LOGO, AP_Amesis Logo:15x15 KiCad QR Code La Boutique Amesis Project, F.Cu at (154.7, 59.7)
- moved   8.35 mm to (98.6, 54.1)

Commit message: PCB prèsque fini (qr  code a modifier
Routing:
- net Net-(G2/G62_OutPut_IAT1-Pad3): track 28.2 -> 29.1 mm
- net Net-(A1-Pad7): track 23.9 -> 24.7 mm
Other:
- board text added: "5v"
- board text added: "CS"
- board text added: "INC"
- board text added: "U/D"
- board text added: "VH"
- board text added: "VL"
- board text added: "VW"

Commit message: Code Arduino Module v0.01 Alfa ok
Parts:
- removed G***: LOGO, AP_Amesis Logo:10x10 KiCad QR Code La Boutique Amesis Project
- removed G***: LOGO, AP_Amesis Logo:15x15 KiCad QR Code La Boutique Amesis Project

Commit message: maj
pcb fini
visu fini
iBom fini HWv.0.01
Parts:
- added  : LOGO, AP_Amesis Logo:15x15 KiCad QR Code La Boutique Amesis Project, F.Cu at (142.0, 54.0)
- added  : LOGO, AP_Amesis Logo:AmesisProject Logo 30mm, B.Cu at (133.7, 52.5)
- added  : LOGO, AP_Amesis Logo:10x10 KiCad QR Code La Boutique Amesis Project, B.Cu at (157.1, 53.3)
- moved G2/G62_OutPut_IAT1 28.7 mm to (141.7, 67.5)
- moved A1 28.7 mm to (157.9, 46.6)
- moved J2 28.7 mm to (164.3, 49.2)
- moved J3 28.7 mm to (149.9, 51.8)
- moved Jumpers_Option1 28.7 mm to (168.5, 46.8)
- moved   28.7 mm to (127.3, 52.3)
- moved G2/G62_InPut_IAT1 28.7 mm to (121.0, 67.5)
- moved IAT_Interne1 28.7 mm to (168.5, 61.5)
- moved J1 28.7 mm to (162.5, 67.5)
Routing:
- net Net-(G2/G62_OutPut_IAT1-Pad3): track 29.1 -> 29.8 mm
Other:
- board text added: "Arduino Nano R3"
- board text added: "No JP = 0 JP 1&2 = + JP 2&3 = ++"
- board text removed: "Arduino Nano"
- board text removed: "Jumper Option Jumper 1&2 = +++ No Jumper = ++ Jumper 2&3 = +"

Commit message: maj pcb et code arduino avec jp et sonde iat
Other:
- board text added: "No JP = 0 JP 1&2 = + JP 2&3 = ++ JP 1&2&3 = +++"
- board text removed: "No JP = 0 JP 1&2 = + JP 2&3 = ++"
Changed lines of the file:
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@@
       (outputformat 1)
       (mirror false)
-      (drillshape 1)
+      (drillshape 0)
       (scaleselection 1)
-      (outputdirectory "")
+      (outputdirectory "012-Amesis-ColdSartE85-backups/Fichier de prod/")
     )
   )
@@
     (effects (font (size 0.8 0.8) (thickness 0.1)))
   )
-  (gr_text " No JP = 0\nJP 1&2 = +\nJP 2&3 = ++" (at 159.005754 58.370904 90) (layer "F.SilkS")
-    (effects (font (size 1 1) (thickness 0.2)) (justify left))
+  (gr_text " No  JP  = 0\nJP  1&2  = +\nJP  2&3  = ++\nJP 1&2&3 = +++" (at 158.9532 57.5564 90) (layer "F.SilkS")
+    (effects (font (size 0.7 0.7) (thickness 0.175)) (justify left))
+  )
+  (dimension (type aligned) (layer "F.Cu")
+    (pts (xy 170.18 44.959704) (xy 118.213354 44.959704))
+    (height 4.827703)
+    (gr_text "51,9666 mm" (at 144.196677 38.332001) (layer "F.Cu")
+      (effects (font (size 1.5 1.5) (thickness 0.3)))
+    )
+    (format (units 3) (units_format 1) (precision 4))
+    (style (thickness 0.2) (arrow_length 1.27) (text_position_mode 0) (extension_height 0.58642) (extension_offset 0.5) keep_text_aligned)
+  )
+  (dimension (type aligned) (layer "F.Cu")
+    (pts (xy 170.300954 71.464104) (xy 170.283354 44.959704))
+    (height 5.484274)
+    (gr_text "26,5044 mm" (at 177.576427 58.207067 -89.96195328) (layer "F.Cu")
+      (effects (font (size 1.5 1.5) (thickness 0.3)))
+    )
+    (format (units 3) (units_format 1) (precision 4))
+    (style (thickness 0.2) (arrow_length 1.27) (text_position_mode 0) (extension_height 0.58642) (extension_offset 0.5) keep_text_aligned)
   )
   (segment (start 151.598954 45.315304) (end 150.268154 46.646104) (width 0.25) (layer "F.Cu") (net 7))

Commit message: code v0.02
termista
Parts:
- removed IAT_Interne1: R_Potentiometer, Connector_PinSocket_2.54mm:PinSocket_1x03_P2.54mm_Vertical
- added R1: R10K, Resistor_THT:R_Axial_DIN0204_L3.6mm_D1.6mm_P5.08mm_Horizontal, F.Cu at (164.2, 62.1)
- added TH1: Thermistor, Connector_PinHeader_2.54mm:PinHeader_1x02_P2.54mm_Vertical, F.Cu at (168.5, 56.4)
Other:
- board text added: "JP 1&2 = +"
- board text added: "JP 1&2&3 = +++"
- board text added: "JP 2&3 = ++"
- board text added: "No JP = 0"
- board text removed: "No JP = 0 JP 1&2 = + JP 2&3 = ++ JP 1&2&3 = +++"
