File: Hardware/Kicad/Laster/012-Amesis-ColdSartE85/012-Amesis-ColdSartE85.kicad_sch (KiCad schematic)
At the start: 8 parts, among them J1 Screw_Terminal_01x02, J2 Conn_01x05_Female, J3 Conn_01x03_Female

Commit message: maj
pcb fini
visu fini
iBom fini HWv.0.01
Changed lines of the file:
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@@
   )
   (symbol (lib_id "Connector:Screw_Terminal_01x02") (at 101.092 29.21 90) (unit 1)
-    (in_bom yes) (on_board yes) (fields_autoplaced)
+    (in_bom yes) (on_board yes)
     (property "Reference" "J1" (id 0) (at 96.52 30.1185 90)
       (effects (font (size 1.27 1.27)) (justify right))
     )
-    (property "Value" "Screw_Terminal_01x02" (id 1) (at 96.52 27.3434 90)
+    (property "Value" "Screw_Terminal_01x02" (id 1) (at 96.266 25.908 90)
       (effects (font (size 1.27 1.27)) (justify right))
     )

Commit message: code v0.02
termista
Parts:
- removed IAT_Interne1: R_Potentiometer, Connector_PinSocket_2.54mm:PinSocket_1x03_P2.54mm_Vertical, symbol Device:R_Potentiometer
- added R1: R10K, Resistor_THT:R_Axial_DIN0204_L3.6mm_D1.6mm_P5.08mm_Horizontal, symbol Device:R
- added TH1: Thermistor, Connector_PinHeader_2.54mm:PinHeader_1x02_P2.54mm_Vertical, symbol Device:Thermistor
Connections:
- net GND: now also R1.2
- net at A1.26 (A7): now also R1.1, TH1.2
- net at A1.27 (+5V), J2.1 (Pin_1): now also TH1.1
Changed lines of the file:
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@@
     (stroke (width 0) (type default) (color 0 0 0 0))
   )
-  (wire (pts (xy 168.402 83.82) (xy 168.402 39.624))
+  (wire (pts (xy 168.402 77.47) (xy 168.402 39.624))
     (stroke (width 0) (type default) (color 0 0 0 0))
   )
@@
     (stroke (width 0) (type default) (color 0 0 0 0))
   )
+  (wire (pts (xy 168.402 97.282) (xy 168.402 95.25))
+    (stroke (width 0) (type default) (color 0 0 0 0))
+  )
   (wire (pts (xy 133.858 97.282) (xy 133.858 95.25))
     (stroke (width 0) (type default) (color 0 0 0 0))
@@
     (stroke (width 0) (type default) (color 0 0 0 0))
   )
-  (wire (pts (xy 146.558 87.63) (xy 164.592 87.63))
+  (wire (pts (xy 146.558 87.63) (xy 168.402 87.63))
     (stroke (width 0) (type default) (color 0 0 0 0))
   )
@@
   )
   (wire (pts (xy 118.11 97.282) (xy 133.858 97.282))
-    (stroke (width 0) (type default) (color 0 0 0 0))
-  )
-  (wire (pts (xy 168.402 91.44) (xy 168.402 97.282))
     (stroke (width 0) (type default) (color 0 0 0 0))
   )
@@
     (pin "3")
     (pin "4")
+  )
+  (symbol (lib_id "Device:R") (at 168.402 91.44 0) (unit 1)
+    (in_bom yes) (on_board yes) (fields_autoplaced)
+    (property "Reference" "R1" (id 0) (at 170.18 90.5315 0)
+      (effects (font (size 1.27 1.27)) (justify left))
+    )
+    (property "Value" "R10K" (id 1) (at 170.18 93.3066 0)
+      (effects (font (size 1.27 1.27)) (justify left))
+    )
+    (property "Footprint" "Resistor_THT:R_Axial_DIN0204_L3.6mm_D1.6mm_P5.08mm_Horizontal" (id 2) (at 166.624 91.44 90)
+      (effects (font (size 1.27 1.27)) hide)
+    )
+    (property "Datasheet" "~" (id 3) (at 168.402 91.44 0)
+      (effects (font (size 1.27 1.27)) hide)
+    )
+    (pin "1")
+    (pin "2")
   )
   (symbol (lib_name "Conn_01x04_Male_1") (lib_id "Connector:Conn_01x04_Male") (at 210.82 73.66 0) (mirror y) (unit 1)
@@
     (pin "3")
   )
-  (symbol (lib_id "Device:R_Potentiometer") (at 168.402 87.63 180) (unit 1)
+  (symbol (lib_id "Device:Thermistor") (at 168.402 82.55 0) (unit 1)
     (in_bom yes) (on_board yes) (fields_autoplaced)
-    (property "Reference" "IAT_Interne1" (id 0) (at 170.18 86.7215 0)
-      (effects (font (size 1.27 1.27)) (justify right))
-    )
-    (property "Value" "R_Potentiometer" (id 1) (at 170.18 89.4966 0)
-      (effects (font (size 1.27 1.27)) (justify right))
-    )
-    (property "Footprint" "Connector_PinSocket_2.54mm:PinSocket_1x03_P2.54mm_Vertical" (id 2) (at 168.402 87.63 0)
-      (effects (font (size 1.27 1.27)) hide)
-    )
-    (property "Datasheet" "~" (id 3) (at 168.402 87.63 0)
-      (effects (font (size 1.27 1.27)) hide)
-    )
-    (pin "1")
-    (pin "2")
-    (pin "3")
+    (property "Reference" "TH1" (id 0) (at 171.069 81.6415 0)
+      (effects (font (size 1.27 1.27)) (justify left))
+    )
+    (property "Value" "Thermistor" (id 1) (at 171.069 84.4166 0)
+      (effects (font (size 1.27 1.27)) (justify left))
+    )
+    (property "Footprint" "Connector_PinHeader_2.54mm:PinHeader_1x02_P2.54mm_Vertical" (id 2) (at 168.402 82.55 0)
+      (effects (font (size 1.27 1.27)) hide)
+    )
+    (property "Datasheet" "~" (id 3) (at 168.402 82.55 0)
+      (effects (font (size 1.27 1.27)) hide)
+    )
+    (pin "1")
+    (pin "2")
   )
   (symbol (lib_name "Conn_01x05_Female_1") (lib_id "Connector:Conn_01x05_Female") (at 104.0892 59.5884 0) (mirror y) (unit 1)
@@
       (reference "G2/G62_OutPut_IAT1") (unit 1) (value "Conn_01x04_Male") (footprint "TerminalBlock:TerminalBlock_bornier-4_P5.08mm")
     )
-    (path "/efe8e9bc-5367-4c16-bae5-490a0bb31048"
-      (reference "IAT_Interne1") (unit 1) (value "R_Potentiometer") (footprint "Connector_PinSocket_2.54mm:PinSocket_1x03_P2.54mm_Vertical")
-    )
     (path "/87d0d2be-75c1-458a-9cdc-395b949ed567"
       (reference "J1") (unit 1) (value "Screw_Terminal_01x02") (footprint "TerminalBlock:TerminalBlock_bornier-2_P5.08mm")
@@
       (reference "Jumpers_Option1") (unit 1) (value "Conn_01x03_Male") (footprint "Connector_PinHeader_2.54mm:PinHeader_1x03_P2.54mm_Vertical")
     )
-  )
+    (path "/3f5ef808-86fd-477c-b6f5-fb0693e0cd9d"
+      (reference "R1") (unit 1) (value "R10K") (footprint "Resistor_THT:R_Axial_DIN0204_L3.6mm_D1.6mm_P5.08mm_Horizontal")
+    )
+    (path "/e1db068e-8ed8-4edf-a7f4-035239f5ddee"
+      (reference "TH1") (unit 1) (value "Thermistor") (footprint "Connector_PinHeader_2.54mm:PinHeader_1x02_P2.54mm_Vertical")
+    )
+  )
