File: Hardware/Kicad/Laster/012-Amesis-ColdSartE85_HWv0.01/012-Amesis-ColdSartE85_HWv0.01.kicad_sch (KiCad schematic)
At the start: 9 parts, among them J1 Screw_Terminal_01x02, J2 Conn_01x05_Female, J3 Conn_01x03_Female

Commit message: maj
Other:
- title: 012-Amesis-ColdStartE85 -> 012-Amesis-ColdStartE85_HW
Changed lines of the file:
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@@
   (paper "A4")
   (title_block
-    (title "012-Amesis-ColdStartE85")
+    (title "012-Amesis-ColdStartE85_HW")
     (date "2022-09-15")
     (rev "v0.01_Golf 1.6L 16v ")
